Commit message: P3 cleanups: Eigen3 dependency, path bandwidth, yaw test, URDF inertials
- Add Eigen3 to the ament_target_dependencies list for consistency
  with the ROS 2 pattern (it is already linked via target_link_libraries).

- Reduce path_max_poses default from 10000 to 1000 to avoid saturating
  DDS bandwidth in networked setups (was ~16.8 MB/s at full capacity).

- Add OppositeWheelRollingIntegratesYaw test that drives left wheels
  forward and right wheels backward, verifying yaw accumulates from
  the contact-solve twist estimate.

- Add placeholder <inertial> elements to all URDF links to silence
  robot_state_publisher warnings and keep the URDF self-contained for
  potential simulation reuse.

File: humble_ws/src/wheel_legged_odometry/urdf/go2w/go2w.urdf (robot description, URDF)
Before this commit: robot go2w, 17 links, 16 joints
Links:
- link FL_calf: mass None -> 0.1
- link FL_hip: mass None -> 0.1
- link FL_thigh: mass None -> 0.1
- link FL_wheel_link: mass None -> 0.1
- link FR_calf: mass None -> 0.1
- link FR_hip: mass None -> 0.1
- link FR_thigh: mass None -> 0.1
- link FR_wheel_link: mass None -> 0.1
- link RL_calf: mass None -> 0.1
- link RL_hip: mass None -> 0.1
- link RL_thigh: mass None -> 0.1
- link RL_wheel_link: mass None -> 0.1
- link RR_calf: mass None -> 0.1
- link RR_hip: mass None -> 0.1
- link RR_thigh: mass None -> 0.1
- link RR_wheel_link: mass None -> 0.1
- link base_link: mass None -> 0.1
